File: ws2812-2020-breakout.kicad_pcb (KiCad board)
At the start: 2 copper layers, 15.6 x 5.5 mm, 6 parts, among them J1 Conn_01x02, J2 Conn_01x02

Commit message: fix
Connections:
- J1 pad 2: Net-(D1-Pad3) -> Net-(D1-Pad2)
- J2 pad 1: Net-(D1-Pad2) -> Net-(D1-Pad3)
Routing:
- net Net-(D1-Pad3): track 3.31 -> 13.3 mm, vias 0 -> 1
- added copper zone on F.Cu, net Net-(D1-Pad2)
- removed copper zone on B.Cu, net Net-(D1-Pad2)
Changed lines of the file:
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@@
     (thickness 1.6)
     (drawings 10)
-    (tracks 10)
+    (tracks 13)
     (zones 0)
     (modules 6)
@@
     (43 Eco2.User user)
     (44 Edge.Cuts user)
-    (45 Margin user)
+    (45 Margin user hide)
     (46 B.CrtYd user hide)
-    (47 F.CrtYd user)
+    (47 F.CrtYd user hide)
     (48 B.Fab user hide)
     (49 F.Fab user hide)
@@
     (pcb_text_size 1.5 1.5)
     (mod_edge_width 0.12)
-    (mod_text_size 1 1)
-    (mod_text_width 0.15)
+    (mod_text_size 0.9144 0.9144)
+    (mod_text_width 0.1524)
     (pad_size 1.7 1.7)
     (pad_drill 1)
@@
       (drillshape 0)
       (scaleselection 1)
-      (outputdirectory "gerber/"))
+      (outputdirectory "gerber"))
   )
   (net 0 "")
@@
     (pad 2 thru_hole oval (at 0 -2.54) (size 1.7 1.7) (drill 1) (layers *.Cu *.Mask)
       (net 7 "Net-(D4-Pad1)"))
-    (pad 1 thru_hole rect (at 0 0) (size 1.7 1.7) (drill 1) (layers *.Cu *.Mask)
-      (net 4 "Net-(D1-Pad2)"))
+    (pad 1 thru_hole circle (at 0 0) (size 1.7 1.7) (drill 1) (layers *.Cu *.Mask)
+      (net 1 "Net-(D1-Pad3)"))
     (model ${KISYS3DMOD}/Connector_PinHeader_2.54mm.3dshapes/PinHeader_1x02_P2.54mm_Vertical.wrl
       (at (xyz 0 0 0))
@@
     (fp_line (start -0.635 1.27) (end 1.27 1.27) (layer B.Fab) (width 0.1))
     (pad 2 thru_hole oval (at 0 -2.54) (size 1.7 1.7) (drill 1) (layers *.Cu *.Mask)
-      (net 1 "Net-(D1-Pad3)"))
-    (pad 1 thru_hole rect (at 0 0) (size 1.7 1.7) (drill 1) (layers *.Cu *.Mask)
+      (net 4 "Net-(D1-Pad2)"))
+    (pad 1 thru_hole circle (at 0 0) (size 1.7 1.7) (drill 1) (layers *.Cu *.Mask)
       (net 2 "Net-(D1-Pad4)"))
     (model ${KISYS3DMOD}/Connector_PinHeader_2.54mm.3dshapes/PinHeader_1x02_P2.54mm_Vertical.wrl
@@
       (net 4 "Net-(D1-Pad2)"))
   )
-  (gr_text "WS2812-2020\nbreakout\ntinyclouds.org" (at 39.3 32.7) (layer B.SilkS)
+  (gr_line (start 47.2 29.7) (end 47.2 35.2) (layer Edge.Cuts) (width 0.05))
+  (gr_text "WS2812-2020\nbreakout\ntinyclouds.org\n" (at 39.3 32.7) (layer B.SilkS)
     (effects (font (size 0.9144 0.9144) (thickness 0.1524)) (justify mirror))
   )
   (gr_line (start 31.6 29.7) (end 31.6 35.2) (layer Edge.Cuts) (width 0.05))
-  (gr_line (start 47.2 29.7) (end 47.2 35.2) (layer Edge.Cuts) (width 0.05))
   (gr_line (start 31.6 35.2) (end 47.2 35.2) (layer Edge.Cuts) (width 0.05))
   (gr_line (start 31.6 29.7) (end 47.2 29.7) (layer Edge.Cuts) (width 0.05))
-  (gr_text GND (at 43 34.6) (layer F.SilkS)
+  (gr_text GND (at 35.31 30.44) (layer F.SilkS)
     (effects (font (size 0.9144 0.9144) (thickness 0.1524)))
   )
@@
     (effects (font (size 0.9144 0.9144) (thickness 0.1524)))
   )
-  (gr_text DO (at 43.4 30.4) (layer F.SilkS)
+  (gr_text DO (at 43.81 30.44) (layer F.SilkS)
     (effects (font (size 0.9144 0.9144) (thickness 0.1524)))
   )
-  (gr_text "DI\n" (at 34.9 30.5) (layer F.SilkS)
+  (gr_text "DI\n" (at 44.04 34.62) (layer F.SilkS)
     (effects (font (size 0.9144 0.9144) (thickness 0.1524)))
   )
-  (gr_text WS2812 (at 39.2 30.4) (layer F.SilkS)
+  (gr_text WS2812 (at 40.07 34.62) (layer F.SilkS)
     (effects (font (size 0.8128 0.8128) (thickness 0.1524)))
   )
-  (segment (start 35.257 33.417) (end 35.4 33.417) (width 0.25) (layer F.Cu) (net 1))
-  (segment (start 33.02 31.18) (end 35.257 33.417) (width 0.25) (layer F.Cu) (net 1))
+  (via blind (at 34.33 32.51) (size 0.45) (drill 0.4) (layers F.Cu B.Cu) (net 1))
+  (segment (start 34.493 32.51) (end 35.4 33.417) (width 0.25) (layer F.Cu) (net 1))
+  (segment (start 34.33 32.51) (end 34.493 32.51) (width 0.25) (layer F.Cu) (net 1))
+  (segment (start 35.475 33.655) (end 34.33 32.51) (width 0.25) (layer B.Cu) (net 1))
+  (segment (start 45.72 33.655) (end 35.475 33.655) (width 0.25) (layer B.Cu) (net 1))
   (segment (start 36.5 32.217) (end 37.7 33.417) (width 0.25) (layer F.Cu) (net 3))
   (segment (start 36.5 31.587) (end 36.5 32.217) (width 0.25) (layer F.Cu) (net 3))
@@
   (segment (start 41.1 32.217) (end 42.3 33.417) (width 0.25) (layer F.Cu) (net 6))
   (segment (start 41.1 31.587) (end 41.1 32.217) (width 0.25) (layer F.Cu) (net 6))
-  (segment (start 45.248 31.587) (end 45.72 31.115) (width 0.25) (layer F.Cu) (net 7))
-  (segment (start 43.4 31.587) (end 45.248 31.587) (width 0.25) (layer F.Cu) (net 7))
-  (zone (net 4) (net_name "Net-(D1-Pad2)") (layer B.Cu) (hatch edge 0.508)
-    (connect_pads (clearance 0.508))
+  (segment (start 43.872 31.115) (end 43.4 31.587) (width 0.25) (layer F.Cu) (net 7))
+  (segment (start 45.72 31.115) (end 43.872 31.115) (width 0.25) (layer F.Cu) (net 7))
+  (zone (net 4) (net_name "Net-(D1-Pad2)") (layer F.Cu) (hatch edge 0.508)
+    (connect_pads yes (clearance 0.508))
     (min_thickness 0.254)
     (fill yes (arc_segments 32) (thermal_gap 0.508) (thermal_bridge_width 0.508))
     (polygon
       (pts
-        (xy 31.6 29.7) (xy 31.6 35.2) (xy 47.2 35.2) (xy 47.2 29.7)
+        (xy 32.7 31.85) (xy 32.7 29.7) (xy 42.7 29.7) (xy 42.7 31.85)
       )
     )
@@
     (polygon
       (pts
-        (xy 31.6 32.8) (xy 31.6 35.2) (xy 44 35.2) (xy 44 32.8)
+        (xy 32.75 35.2) (xy 32.75 33.05) (xy 43.7 33.025) (xy 43.7 35.175)
       )
     )
